Commit message: Change SLAM to Localization

File: description/robot_core.xacro (robot description, xacro)
@@ -20,11 +20,11 @@
     <!-- Create Robot BASE LINK -->
     <link name="base_link"></link>
-    <!-- Create Robot BASE FOOT PRINT -->
+    <!-- Create Robot BASE FOOTPRINT -->
     <joint name="base_footprint_joint" type="fixed">
         <parent link="base_link"/>
-        <child link="base_footprint_link"/>
+        <child link="base_footprint"/>
         <origin xyz="0 0 0" rpy="0 0 0"/>
     </joint>
-    <link name="base_footprint_link"></link>
+    <link name="base_footprint"></link>
     <!-- Create Robot CHASSIS LINK and JOINT with BASE LINK -->
     <joint name="chassis_joint" type="fixed">
