Commit message: Adding Robot Meshes

File: description/lidar.xacro (robot description, xacro)
@@ -50,5 +50,5 @@
             <plugin name="laser_controller" filename="libgazebo_ros_ray_sensor.so">
                 <ros>
-                    <argument>~/out:=scan</argument>
+                    <argument>~/out:=scan2</argument>
                 </ros>
                 <output_type>sensor_msgs/LaserScan</output_type>

File: description/robot_core.xacro (robot description, xacro)
@@ -31,4 +31,5 @@
             <geometry>
                 <box size="0.3 0.3 0.15"/>
+                <!-- <mesh filename="package://my_bot/meshes/AGV-Body-Cut.stl"/> -->
             </geometry>
             <material name="white"/>

Commit message: Adding SLAM

File: description/lidar.xacro (robot description, xacro)
@@ -50,5 +50,5 @@
             <plugin name="laser_controller" filename="libgazebo_ros_ray_sensor.so">
                 <ros>
-                    <argument>~/out:=scan2</argument>
+                    <argument>~/out:=scan</argument>
                 </ros>
                 <output_type>sensor_msgs/LaserScan</output_type>

File: description/robot_core.xacro (robot description, xacro)
@@ -20,4 +20,11 @@
     <!-- Create Robot BASE LINK -->
     <link name="base_link"></link>
+    <!-- Create Robot BASE FOOT PRINT -->
+    <joint name="base_footprint_joint" type="fixed">
+        <parent link="base_link"/>
+        <child link="base_footprint_link"/>
+        <origin xyz="0 0 0" rpy="0 0 0"/>
+    </joint>
+    <link name="base_footprint_link"></link>
     <!-- Create Robot CHASSIS LINK and JOINT with BASE LINK -->
     <joint name="chassis_joint" type="fixed">

Commit message: Tweaking ROS Control

File: description/lidar.xacro (robot description, xacro)
@@ -33,5 +33,5 @@
         <sensor name="laser" type="ray">
             <pose> 0 0 0 0 0 0 </pose>
-            <visualize>true</visualize>
+            <visualize>false</visualize>
             <update_rate>10</update_rate>
             <ray>

File: description/robot.urdf.xacro (robot description, xacro)
@@ -1,7 +1,12 @@
 <?xml version="1.0"?>
 <robot xmlns:xacro="http://www.ros.org/wiki/xacro"  name="robot">
+    <xacro:arg name="use_ros2_control" default="true"/>
     <xacro:include filename="robot_core.xacro"/>
-    <!-- <xacro:include filename="gazebo_control.xacro"/> -->
-    <xacro:include filename="ros2_control.xacro"/>
+    <xacro:if value="$(arg use_ros2_control)">
+        <xacro:include filename="ros2_control.xacro"/>
+    </xacro:if>
+    <xacro:unless value="$(arg use_ros2_control)">
+        <xacro:include filename="gazebo_control.xacro"/>
+    </xacro:unless>
     <xacro:include filename="lidar.xacro"/>
 </robot>

File: description/robot_core.xacro (robot description, xacro)
@@ -72,5 +72,6 @@
         <collision>
             <geometry>
-                <cylinder radius="0.05" length="0.04"/>
+                <!-- <cylinder radius="0.05" length="0.04"/> -->
+                <sphere radius="0.05"/>
             </geometry>
             <material name="blue"/>
@@ -99,5 +100,6 @@
         <collision>
             <geometry>
-                <cylinder radius="0.05" length="0.04"/>
+                <!-- <cylinder radius="0.05" length="0.04"/> -->
+                <sphere radius="0.05"/>
             </geometry>
             <material name="blue"/>
